File: adapter/spiflash.kicad_pcb (KiCad board)
At the start: 2 copper layers, 35 x 22 mm, 46 parts, among them J1 USB_C_Receptacle_USB2.0, J2 Tag-Connect, J3 Conn_01x02, J4 Conn_01x03, J5 Clip, U1 XC6206, U2 SRV05-4-P-T7, U4 STM32F103C8T6, U5 SN74LVC1T45DBV, U6 SN74LVC1T45DBV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

Commit message: adapter: define crystal loading caps, reexport fab
Parts:
- C3, C6: value TBD -> 20p
Changed lines of the file:
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@@
       (effects (font (size 1 1) (thickness 0.15)))
     )
-    (fp_text value TBD (at 0 1.17 90) (layer F.Fab)
+    (fp_text value 20p (at 0 1.17 90) (layer F.Fab)
       (effects (font (size 1 1) (thickness 0.15)))
     )
@@
       (effects (font (size 1 1) (thickness 0.15)))
     )
-    (fp_text value TBD (at 0 1.17 90) (layer F.Fab)
+    (fp_text value 20p (at 0 1.17 90) (layer F.Fab)
       (effects (font (size 1 1) (thickness 0.15)))
     )
