File: breakout/so8.sch (KiCad schematic (older format))
At the start: 3 parts, among them J1 Conn_02x04_Odd_Even, U1 W25Q32JVSS

Commit message: breakout: add PWR_FLAGs
Add PWR_FLAGs to the supply lines to silence ERC warnings.

Fixes #2.
Connections:
- wire segments 22 -> 24
Changed lines of the file:
@@
 Wire Wire Line
 	6750 3600 6700 3600
+$Comp
+L power:VCC #PWR?
+U 1 1 5E069067
+P 7350 3150
+F 0 "#PWR?" H 7350 3000 50  0001 C CNN
+F 1 "VCC" H 7367 3323 50  0000 C CNN
+F 2 "" H 7350 3150 50  0001 C CNN
+F 3 "" H 7350 3150 50  0001 C CNN
+	1    7350 3150
+	1    0    0    -1
+$EndComp
+$Comp
+L power:GND #PWR?
+U 1 1 5E06937F
+P 7700 3200
+F 0 "#PWR?" H 7700 2950 50  0001 C CNN
+F 1 "GND" H 7705 3027 50  0000 C CNN
+F 2 "" H 7700 3200 50  0001 C CNN
+F 3 "" H 7700 3200 50  0001 C CNN
+	1    7700 3200
+	1    0    0    -1
+$EndComp
+$Comp
+L power:PWR_FLAG #FLG?
+U 1 1 5E0698C6
+P 7700 3150
+F 0 "#FLG?" H 7700 3225 50  0001 C CNN
+F 1 "PWR_FLAG" H 7700 3323 50  0000 C CNN
+F 2 "" H 7700 3150 50  0001 C CNN
+F 3 "~" H 7700 3150 50  0001 C CNN
+	1    7700 3150
+	1    0    0    -1
+$EndComp
+Wire Wire Line
+	7700 3150 7700 3200
+Wire Wire Line
+	7350 3200 7350 3150
+$Comp
+L power:PWR_FLAG #FLG?
+U 1 1 5E06A7DA
+P 7350 3200
+F 0 "#FLG?" H 7350 3275 50  0001 C CNN
+F 1 "PWR_FLAG" H 7350 3373 50  0000 C CNN
+F 2 "" H 7350 3200 50  0001 C CNN
+F 3 "~" H 7350 3200 50  0001 C CNN
+	1    7350 3200
+	-1   0    0    1
+$EndComp
 $EndSCHEMATC
